File: Episode05/DTypeEdgeTriggered/DTypeEdgeTriggered.sch (KiCad schematic (older format))
At the start: 18 parts, among them SW1 SW_Push, SW2 SW_Push, U1 74HC00, U2 74HC00, U3 74HC00, U4 74HC14

Commit message: fix switch debouncing
For this circuit, the Schmitt trigger inverters are
supposed to go high when the button is pressed, not low.
Connections:
- net GND: now also C1.2, C2.2, SW1.1, SW2.1; no longer R1.2, R2.2
- net VCC: now also R1.1, R2.1; no longer C1.1, C2.1, SW1.1, SW2.1
- net at SW1.2, U4.1: now also C1.1, R1.2; no longer C1.2, R1.1
- net at SW2.2, U4.3: now also C2.1, R2.2; no longer C2.2, R2.1
Other:
- moved on the sheet: C1, R1
Changed lines of the file:
@@
 	1600 1400 1500 1400
 Wire Wire Line
-	1500 1400 1500 850
-$Comp
-L power:VCC #PWR?
-U 1 1 5C5F5D6A
-P 1500 850
-F 0 "#PWR?" H 1500 700 50  0001 C CNN
-F 1 "VCC" H 1517 1023 50  0000 C CNN
-F 2 "" H 1500 850 50  0001 C CNN
-F 3 "" H 1500 850 50  0001 C CNN
-	1    1500 850
-	1    0    0    -1
-$EndComp
+	1500 1400 1500 2300
 Wire Wire Line
 	2100 1400 2100 1850
@@
 L device:R R1
 U 1 1 5C5FA310
-P 2100 2000
-F 0 "R1" H 2170 2046 50  0000 L CNN
-F 1 "30K" H 2170 1955 50  0000 L CNN
-F 2 "" V 2030 2000 50  0001 C CNN
-F 3 "" H 2100 2000 50  0001 C CNN
-	1    2100 2000
+P 2100 1100
+F 0 "R1" H 2170 1146 50  0000 L CNN
+F 1 "30K" H 2170 1055 50  0000 L CNN
+F 2 "" V 2030 1100 50  0001 C CNN
+F 3 "" H 2100 1100 50  0001 C CNN
+	1    2100 1100
 	1    0    0    -1
 $EndComp
@@
 $EndComp
 $Comp
-L Switch:SW_Push SW2
-U 1 1 5C6272AB
-P 4250 1400
-F 0 "SW2" H 4250 1685 50  0000 C CNN
-F 1 "SW_Push" H 4250 1594 50  0000 C CNN
-F 2 "" H 4250 1600 50  0001 C CNN
-F 3 "" H 4250 1600 50  0001 C CNN
-	1    4250 1400
-	1    0    0    -1
-$EndComp
-Wire Wire Line
-	4050 1400 3950 1400
-Wire Wire Line
-	3950 1400 3950 850
-$Comp
-L power:VCC #PWR?
-U 1 1 5C6272BB
-P 3950 850
-F 0 "#PWR?" H 3950 700 50  0001 C CNN
-F 1 "VCC" H 3967 1023 50  0000 C CNN
-F 2 "" H 3950 850 50  0001 C CNN
-F 3 "" H 3950 850 50  0001 C CNN
-	1    3950 850
-	1    0    0    -1
-$EndComp
-Wire Wire Line
-	4550 1400 4550 1850
-$Comp
-L device:R R2
-U 1 1 5C6272C2
-P 4550 2000
-F 0 "R2" H 4620 2046 50  0000 L CNN
-F 1 "30K" H 4620 1955 50  0000 L CNN
-F 2 "" V 4480 2000 50  0001 C CNN
-F 3 "" H 4550 2000 50  0001 C CNN
-	1    4550 2000
-	1    0    0    -1
-$EndComp
-Wire Wire Line
-	4550 2150 4550 2300
-$Comp
-L power:GND #PWR?
-U 1 1 5C6272CA
-P 4550 2300
-F 0 "#PWR?" H 4550 2050 50  0001 C CNN
-F 1 "GND" H 4555 2127 50  0000 C CNN
-F 2 "" H 4550 2300 50  0001 C CNN
-F 3 "" H 4550 2300 50  0001 C CNN
-	1    4550 2300
-	1    0    0    -1
-$EndComp
-Wire Wire Line
-	4450 1400 4550 1400
-Wire Wire Line
-	4750 1400 4550 1400
-Connection ~ 4550 1400
-$Comp
-L power:VCC #PWR?
-U 1 1 5C6272D4
-P 4550 850
-F 0 "#PWR?" H 4550 700 50  0001 C CNN
-F 1 "VCC" H 4567 1023 50  0000 C CNN
-F 2 "" H 4550 850 50  0001 C CNN
-F 3 "" H 4550 850 50  0001 C CNN
-	1    4550 850
-	1    0    0    -1
-$EndComp
-$Comp
 L device:LED D2
 U 1 1 5C6272DA
@@
 L device:C C1
 U 1 1 5C6639B7
-P 2100 1100
-F 0 "C1" H 2215 1146 50  0000 L CNN
-F 1 "0.1uF" H 2215 1055 50  0000 L CNN
-F 2 "" H 2138 950 50  0001 C CNN
-F 3 "" H 2100 1100 50  0001 C CNN
-	1    2100 1100
+P 2100 2000
+F 0 "C1" H 2215 2046 50  0000 L CNN
+F 1 "0.1uF" H 2215 1955 50  0000 L CNN
+F 2 "" H 2138 1850 50  0001 C CNN
+F 3 "" H 2100 2000 50  0001 C CNN
+	1    2100 2000
 	1    0    0    -1
 $EndComp
@@
 Wire Wire Line
 	2100 1250 2100 1400
-$Comp
-L device:C C2
-U 1 1 5C66B94A
-P 4550 1100
-F 0 "C2" H 4665 1146 50  0000 L CNN
-F 1 "0.1uF" H 4665 1055 50  0000 L CNN
-F 2 "" H 4588 950 50  0001 C CNN
-F 3 "" H 4550 1100 50  0001 C CNN
-	1    4550 1100
-	1    0    0    -1
-$EndComp
-Wire Wire Line
-	4550 850  4550 950
-Wire Wire Line
-	4550 1250 4550 1400
 $Comp
 L 74xx:74HC14 U4
@@
 Wire Wire Line
 	8950 4550 10250 4550
+$Comp
+L power:GND #PWR?
+U 1 1 5C603161
+P 1500 2300
+F 0 "#PWR?" H 1500 2050 50  0001 C CNN
+F 1 "GND" H 1505 2127 50  0000 C CNN
+F 2 "" H 1500 2300 50  0001 C CNN
+F 3 "" H 1500 2300 50  0001 C CNN
+	1    1500 2300
+	1    0    0    -1
+$EndComp
+$Comp
+L Switch:SW_Push SW2
+U 1 1 5C608100
+P 4250 1400
+F 0 "SW2" H 4250 1685 50  0000 C CNN
+F 1 "SW_Push" H 4250 1594 50  0000 C CNN
+F 2 "" H 4250 1600 50  0001 C CNN
+F 3 "" H 4250 1600 50  0001 C CNN
+	1    4250 1400
+	1    0    0    -1
+$EndComp
+Wire Wire Line
+	4050 1400 3950 1400
+Wire Wire Line
+	3950 1400 3950 2300
+Wire Wire Line
+	4550 1400 4550 1850
+$Comp
+L device:R R2
+U 1 1 5C60810A
+P 4550 1100
+F 0 "R2" H 4620 1146 50  0000 L CNN
+F 1 "30K" H 4620 1055 50  0000 L CNN
+F 2 "" V 4480 1100 50  0001 C CNN
+F 3 "" H 4550 1100 50  0001 C CNN
+	1    4550 1100
+	1    0    0    -1
+$EndComp
+Wire Wire Line
+	4550 2150 4550 2300
+$Comp
+L power:GND #PWR?
+U 1 1 5C608112
+P 4550 2300
+F 0 "#PWR?" H 4550 2050 50  0001 C CNN
+F 1 "GND" H 4555 2127 50  0000 C CNN
+F 2 "" H 4550 2300 50  0001 C CNN
+F 3 "" H 4550 2300 50  0001 C CNN
+	1    4550 2300
+	1    0    0    -1
+$EndComp
+Wire Wire Line
+	4450 1400 4550 1400
+Wire Wire Line
+	4750 1400 4550 1400
+Connection ~ 4550 1400
+$Comp
+L power:VCC #PWR?
+U 1 1 5C60811B
+P 4550 850
+F 0 "#PWR?" H 4550 700 50  0001 C CNN
+F 1 "VCC" H 4567 1023 50  0000 C CNN
+F 2 "" H 4550 850 50  0001 C CNN
+F 3 "" H 4550 850 50  0001 C CNN
+	1    4550 850
+	1    0    0    -1
+$EndComp
+$Comp
+L device:C C2
+U 1 1 5C608121
+P 4550 2000
+F 0 "C2" H 4665 2046 50  0000 L CNN
+F 1 "0.1uF" H 4665 1955 50  0000 L CNN
+F 2 "" H 4588 1850 50  0001 C CNN
+F 3 "" H 4550 2000 50  0001 C CNN
+	1    4550 2000
+	1    0    0    -1
+$EndComp
+Wire Wire Line
+	4550 850  4550 950
+Wire Wire Line
+	4550 1250 4550 1400
+$Comp
+L power:GND #PWR?
+U 1 1 5C60812A
+P 3950 2300
+F 0 "#PWR?" H 3950 2050 50  0001 C CNN
+F 1 "GND" H 3955 2127 50  0000 C CNN
+F 2 "" H 3950 2300 50  0001 C CNN
+F 3 "" H 3950 2300 50  0001 C CNN
+	1    3950 2300
+	1    0    0    -1
+$EndComp
 $EndSCHEMATC
