File: Episode05/SRLatch/SRLatch.sch (KiCad schematic (older format))
At the start: 16 parts, among them SW1 SW_Push, SW2 SW_Push, U1 74HC14, U2 74HC00

Commit message: label -S and -R inputs correctly
Connections:
- net R renamed -S
- net S renamed -R
Changed lines of the file:
@@
 EESchema Schematic File Version 4
+LIBS:SRLatch-cache
 EELAYER 26 0
 EELAYER END
@@
 Wire Wire Line
 	5100 4200 5100 1750
-Text Label 6250 3050 0    50   ~ 0
-R
-Text Label 6250 4200 0    50   ~ 0
-S
 $Comp
 L device:R R5
@@
 	6100 6350 5650 6350
 Connection ~ 5650 6350
+Text Label 6200 3050 0    50   ~ 0
+-S
+Text Label 6200 4200 0    50   ~ 0
+-R
 $EndSCHEMATC
