File: Episode05/DTypeLatch/DTypeLatch.sch (KiCad schematic (older format))
At the start: 18 parts, among them SW1 SW_Push, SW2 SW_Push, U1 74HC14, U2 74HC00, U3 74HC00

Commit message: added missing component designations
Parts:
- gave numbers to parts that had none: 2
Changed lines of the file:
@@
 $EndComp
 $Comp
-L device:C C?
+L device:C C1
 U 1 1 5C5F0D10
 P 1250 2250
-F 0 "C?" H 1365 2296 50  0000 L CNN
+F 0 "C1" H 1365 2296 50  0000 L CNN
 F 1 "0.1uF" H 1365 2205 50  0000 L CNN
 F 2 "" H 1288 2100 50  0001 C CNN
@@
 $EndComp
 $Comp
-L device:C C?
+L device:C C2
 U 1 1 5C5F1BA3
 P 3400 2250
-F 0 "C?" H 3515 2296 50  0000 L CNN
+F 0 "C2" H 3515 2296 50  0000 L CNN
 F 1 "0.1uF" H 3515 2205 50  0000 L CNN
 F 2 "" H 3438 2100 50  0001 C CNN
