File: Episode0d/CircuitWithPeriphs/CPUandGlueLogic.sch (KiCad schematic (older format))
At the start: 27 parts, among them SW100 SW_Push, U100 74HCT245, U101 74HCT245, U102 MAX708, U103 HD6809, U104 74HCT245, U105 74HCT365, U106 74HCT00, U107 74HCT27, U108 74HCT138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

Commit message: working on integrating ACIA device
Connections:
- wire segments 323 -> 322
Changed lines of the file:
@@
 	1    0    0    -1
 $EndComp
-Wire Wire Line
-	5250 7150 5250 7250
-$Comp
-L power:GND #PWR?
-U 1 1 5DC72C2F
-P 5250 7250
-F 0 "#PWR?" H 5250 7000 50  0001 C CNN
-F 1 "GND" H 5255 7077 50  0000 C CNN
-F 2 "" H 5250 7250 50  0001 C CNN
-F 3 "" H 5250 7250 50  0001 C CNN
-	1    5250 7250
-	1    0    0    -1
-$EndComp
+Text Label 5350 7150 0    50   ~ 0
+R~W
 Wire Bus Line
 	1000 5700 3650 5700
@@
 Wire Bus Line
 	2450 6150 2450 9200
+Text HLabel 6850 7150 2    50   Output ~ 0
+R~W
 $EndSCHEMATC
