File: Episode12/CircuitWithKbdCtrl/Keyboard.sch (KiCad schematic (older format))
At the start: 13 parts, among them J501 Conn_01x20, U501 87C51/89C51, U502 IDT7201, U503 74LS138, U504 74HCT541, Y501 11.0592 MHz

Commit message: '138 device is 74HCT138, not 74LS138
Parts:
- U503: value 74LS138 -> 74HCT138
Changed lines of the file:
@@
 P 5550 1600
 F 0 "U503" H 5550 2381 50  0000 C CNN
-F 1 "74LS138" H 5550 2290 50  0000 C CNN
+F 1 "74HCT138" H 5550 2290 50  0000 C CNN
 F 2 "" H 5550 1600 50  0001 C CNN
 F 3 "" H 5550 1600 50  0001 C CNN
@@
 	2850 5800 3050 5800
 NoConn ~ 3050 5800
+Text Notes 2100 6300 0    50   ~ 0
+Note that RN501 could also be\na 9 pin (8 resistor) network.\nThe exact value isn't critical:\nanything between 2k7 and 47k\nshould work fine.
 Wire Bus Line
 	7150 1550 7150 4900
 Wire Bus Line
 	9800 1550 9800 6550
-Text Notes 2100 6300 0    50   ~ 0
-Note that RN501 could also be\na 9 pin (8 resistor) network.\nThe exact value isn't critical:\nanything between 2k7 and 47k\nshould work fine.
 $EndSCHEMATC
