File: HardwareDesign/Interrupts.sch (KiCad schematic (older format))
At the start: 21 parts, among them U401 74HCT74, U402 74HCT11, U403 74HCT147, U404 74HCT540, U405 74HCT574, U406 74HCT32, U407 74HCT32

Commit message: more cleanups in preparation for PCB layout
Renamed nets to distinguish unbuffered vs. buffered signals.

Fixed one error in interrupt controller (D0 was tied
to ground.)

Not entirely done yet.
Connections:
- net GND: no longer U404.18 (Y0)
- new net D0: U404.18 (Y0)
Changed lines of the file:
@@
 Wire Wire Line
 	2050 6050 1400 6050
-Text Label 1900 5350 0    50   ~ 0
-D0
 Text Label 1900 5450 0    50   ~ 0
 D1

Commit message: more preparations for PCB layout
Make sure all nets connected to backplane connector pins are
labeled correctly.

Add bulk decoupling caps for each backplane connector.

Make keyboard interrupt be -IRQ5 rather than -IRQ7.
Changed lines of the file:
@@
 	2950 7500 2950 6950
 Wire Bus Line
-	1400 7050 3050 7050
+	1400 7050 3500 7050
 Entry Bus Bus
 	1300 6950 1400 7050
@@
 	6950 2100 8250 2100
 Entry Bus Bus
-	3050 7050 3150 6950
+	3500 7050 3600 6950
 Wire Bus Line
-	3150 6950 3150 6700
+	3600 6950 3600 6700
 Entry Bus Bus
-	3150 6700 3250 6600
+	3600 6700 3700 6600
 Wire Bus Line
-	3250 6600 10250 6600
+	3700 6600 10250 6600
 Entry Bus Bus
 	10250 6600 10350 6500

Commit message: a few more consistency tweaks before PCB layout
Routed second timer/counter output to backplane connector,
just in case we want to use it for something eventually
Parts:
- C401, C402, C403, C404, C405, C406, C407: value 100nF -> 0.1 μF
Changed lines of the file:
@@
 P 650 8250
 F 0 "C401" H 765 8296 50  0000 L CNN
-F 1 "100nF" H 765 8205 50  0000 L CNN
+F 1 "0.1 μF" H 765 8205 50  0000 L CNN
 F 2 "" H 688 8100 50  0001 C CNN
 F 3 "" H 650 8250 50  0001 C CNN
 	1    650  8250
-	1    0    0    -1
-$EndComp
-$Comp
-L device:C C402
-U 1 1 5E1B7F4B
-P 1150 8250
-F 0 "C402" H 1265 8296 50  0000 L CNN
-F 1 "100nF" H 1265 8205 50  0000 L CNN
-F 2 "" H 1188 8100 50  0001 C CNN
-F 3 "" H 1150 8250 50  0001 C CNN
-	1    1150 8250
-	1    0    0    -1
-$EndComp
-$Comp
-L device:C C403
-U 1 1 5E1BBD0D
-P 1650 8250
-F 0 "C403" H 1765 8296 50  0000 L CNN
-F 1 "100nF" H 1765 8205 50  0000 L CNN
-F 2 "" H 1688 8100 50  0001 C CNN
-F 3 "" H 1650 8250 50  0001 C CNN
-	1    1650 8250
-	1    0    0    -1
-$EndComp
-$Comp
-L device:C C404
-U 1 1 5E1BBD13
-P 2150 8250
-F 0 "C404" H 2265 8296 50  0000 L CNN
-F 1 "100nF" H 2265 8205 50  0000 L CNN
-F 2 "" H 2188 8100 50  0001 C CNN
-F 3 "" H 2150 8250 50  0001 C CNN
-	1    2150 8250
 	1    0    0    -1
 $EndComp
@@
 Text Label 10000 4850 0    50   ~ 0
 D7
-$Comp
-L device:C C405
-U 1 1 5E75B086
-P 2600 8250
-F 0 "C405" H 2715 8296 50  0000 L CNN
-F 1 "100nF" H 2715 8205 50  0000 L CNN
-F 2 "" H 2638 8100 50  0001 C CNN
-F 3 "" H 2600 8250 50  0001 C CNN
-	1    2600 8250
-	1    0    0    -1
-$EndComp
-$Comp
-L device:C C406
-U 1 1 5E75B08C
-P 3100 8250
-F 0 "C406" H 3215 8296 50  0000 L CNN
-F 1 "100nF" H 3215 8205 50  0000 L CNN
-F 2 "" H 3138 8100 50  0001 C CNN
-F 3 "" H 3100 8250 50  0001 C CNN
-	1    3100 8250
-	1    0    0    -1
-$EndComp
-$Comp
-L device:C C407
-U 1 1 5E75B092
-P 3600 8250
-F 0 "C407" H 3715 8296 50  0000 L CNN
-F 1 "100nF" H 3715 8205 50  0000 L CNN
-F 2 "" H 3638 8100 50  0001 C CNN
-F 3 "" H 3600 8250 50  0001 C CNN
-	1    3600 8250
-	1    0    0    -1
-$EndComp
 Wire Wire Line
 	3100 8100 3100 8000
@@
 	1700 5350 1700 6350
 Connection ~ 1700 6350
+$Comp
+L device:C C402
+U 1 1 611239CC
+P 1150 8250
+F 0 "C402" H 1265 8296 50  0000 L CNN
+F 1 "0.1 μF" H 1265 8205 50  0000 L CNN
+F 2 "" H 1188 8100 50  0001 C CNN
+F 3 "" H 1150 8250 50  0001 C CNN
+	1    1150 8250
+	1    0    0    -1
+$EndComp
+$Comp
+L device:C C403
+U 1 1 611393F5
+P 1650 8250
+F 0 "C403" H 1765 8296 50  0000 L CNN
+F 1 "0.1 μF" H 1765 8205 50  0000 L CNN
+F 2 "" H 1688 8100 50  0001 C CNN
+F 3 "" H 1650 8250 50  0001 C CNN
+	1    1650 8250
+	1    0    0    -1
+$EndComp
+$Comp
+L device:C C404
+U 1 1 61139593
+P 2150 8250
+F 0 "C404" H 2265 8296 50  0000 L CNN
+F 1 "0.1 μF" H 2265 8205 50  0000 L CNN
+F 2 "" H 2188 8100 50  0001 C CNN
+F 3 "" H 2150 8250 50  0001 C CNN
+	1    2150 8250
+	1    0    0    -1
+$EndComp
+$Comp
+L device:C C405
+U 1 1 6114FB2B
+P 2600 8250
+F 0 "C405" H 2715 8296 50  0000 L CNN
+F 1 "0.1 μF" H 2715 8205 50  0000 L CNN
+F 2 "" H 2638 8100 50  0001 C CNN
+F 3 "" H 2600 8250 50  0001 C CNN
+	1    2600 8250
+	1    0    0    -1
+$EndComp
+$Comp
+L device:C C406
+U 1 1 6114FDA9
+P 3100 8250
+F 0 "C406" H 3215 8296 50  0000 L CNN
+F 1 "0.1 μF" H 3215 8205 50  0000 L CNN
+F 2 "" H 3138 8100 50  0001 C CNN
+F 3 "" H 3100 8250 50  0001 C CNN
+	1    3100 8250
+	1    0    0    -1
+$EndComp
+$Comp
+L device:C C407
+U 1 1 6114FDB3
+P 3600 8250
+F 0 "C407" H 3715 8296 50  0000 L CNN
+F 1 "0.1 μF" H 3715 8205 50  0000 L CNN
+F 2 "" H 3638 8100 50  0001 C CNN
+F 3 "" H 3600 8250 50  0001 C CNN
+	1    3600 8250
+	1    0    0    -1
+$EndComp
 Wire Bus Line
 	10350 4250 10350 6500

Commit message: changes to backplane signals
Route all IRQ signals on backplane.

Only route -IOR1..-IOR3 on backplane.

Move TCOUNT2 to after IRQ signals.
Connections:
- net ~IRQ3 renamed IRQ3
- net IRQ3: no longer U401.5 (Q), U406.9
- net ~IRQ6 renamed IRQ6
- net IRQ6: no longer U401.9 (Q), U407.4
- new net ~IRQ3~: U401.5 (Q), U406.9
- new net ~IRQ6~: U401.9 (Q), U407.4
Other:
- note added: "IRQ3_IN and IRQ6_IN are\nedge-triggered (positive\nedge)\n\n~IRQ3_CLR~ and ~IRQ6_CLR~\ncan be temporarily\nasserted to clear ~IRQ3~/\n~IRQ6~ after they are\ntriggered"
- note removed: "~IRQ3_IN~ and ~IRQ6_IN~ are\nedge-triggered (positive\nedge)\n\n~IRQ3_CLR~ and ~IRQ6_CLR~\ncan be temporarily\nasserted to clear ~IRQ3~/\n~IRQ6~ after they are\ntriggered"
Changed lines of the file:
@@
 ~IRQ7
 Text Notes 750  1300 0    50   ~ 0
-~IRQ3_IN~ and ~IRQ6_IN~ are\nedge-triggered (positive\nedge)\n\n~IRQ3_CLR~ and ~IRQ6_CLR~\ncan be temporarily\nasserted to clear ~IRQ3~/\n~IRQ6~ after they are\ntriggered
+IRQ3_IN and IRQ6_IN are\nedge-triggered (positive\nedge)\n\n~IRQ3_CLR~ and ~IRQ6_CLR~\ncan be temporarily\nasserted to clear ~IRQ3~/\n~IRQ6~ after they are\ntriggered
 Text HLabel 1100 1650 0    50   Input ~ 0
-~IRQ3
+IRQ3
 Text HLabel 1100 1950 0    50   Input ~ 0
-~IRQ6
+IRQ6
 $Comp
 L device:R R401
@@
 ~IRQ5_IN
 Text Label 1200 1950 0    50   ~ 0
-~IRQ6_IN
+IRQ6_IN
 Text Label 3750 2050 0    50   ~ 0
 ~IRQ7
@@
 ~IRQ2
 Text Label 3750 1650 0    50   ~ 0
-~IRQ3
+~IRQ3~
 Text Label 3750 1750 0    50   ~ 0
 ~IRQ4
@@
 ~IRQ5
 Text Label 3750 1950 0    50   ~ 0
-~IRQ6
+~IRQ6~
 Text Label 1200 2050 0    50   ~ 0
 ~IRQ7_IN
@@
 	2000 1650 1100 1650
 Text Label 1200 1650 0    50   ~ 0
-~IRQ3_IN
+IRQ3_IN
 Wire Wire Line
 	1650 4050 1650 1950

Commit message: assigned component footprints
Parts:
- C401, C402, C403, C404, C405, C406, C407: footprint (none) -> Capacitor_THT:C_Disc_D5.0mm_W2.5mm_P2.50mm
- R401, R402, R403, R404, R405, R406, R407: footprint (none) -> Resistor_THT:R_Axial_DIN0204_L3.6mm_D1.6mm_P7.62mm_Horizontal
- U401, U402, U406, U407: footprint (none) -> Package_DIP:DIP-14_W7.62mm_Socket
- U403: footprint (none) -> Package_DIP:DIP-16_W7.62mm_Socket
- U404, U405: footprint (none) -> Package_DIP:DIP-20_W7.62mm_Socket
