File: HardwareDesign/Keyboard.sch (KiCad schematic (older format))
At the start: 14 parts, among them J501 Conn_01x20, J503 Conn_01x02, U501 87C51/89C51, U502 IDT7201, U503 74HCT138, U504 74HCT541, Y501 11.0592 MHz

Commit message: assigned component footprints
Parts:
- C501, C502, C503, C504: footprint (none) -> Capacitor_THT:C_Disc_D5.0mm_W2.5mm_P2.50mm
- C505, C506: footprint (none) -> Capacitor_THT:C_Disc_D3.8mm_W2.6mm_P2.50mm
- J501: footprint (none) -> Connector_PinHeader_2.54mm:PinHeader_1x20_P2.54mm_Vertical
- J503: footprint (none) -> Connector_PinHeader_2.54mm:PinHeader_1x02_P2.54mm_Vertical
- U501: footprint DIP254P1524X470-40 -> Package_DIP:DIP-40_W15.24mm_Socket
- U502: footprint (none) -> Package_DIP:DIP-28_W7.62mm_Socket
- U503: footprint (none) -> Package_DIP:DIP-16_W7.62mm_Socket
- U504: footprint (none) -> Package_DIP:DIP-20_W7.62mm_Socket
- Y501: footprint (none) -> Crystal:Crystal_HC18-U_Vertical
Changed lines of the file:
@@
 F 0 "U502" H 8150 3231 50  0000 C CNN
 F 1 "IDT7201" H 8150 3140 50  0000 C CNN
-F 2 "" H 8150 2050 50  0001 C CNN
+F 2 "Package_DIP:DIP-28_W7.62mm_Socket" H 8150 2050 50  0001 C CNN
 F 3 "" H 8150 2050 50  0001 C CNN
 	1    8150 2050
@@
 F 0 "U501" H 4450 6720 50  0000 C CNN
 F 1 "87C51/89C51" H 4450 6629 50  0000 C CNN
-F 2 "DIP254P1524X470-40" H 4450 4950 50  0001 L BNN
+F 2 "Package_DIP:DIP-40_W15.24mm_Socket" H 4450 4950 50  0001 L BNN
 F 3 "None" H 4450 4950 50  0001 L BNN
 F 4 "NXP Semiconductors" H 4450 4950 50  0001 L BNN "Field4"
@@
 F 0 "U503" H 5100 2431 50  0000 C CNN
 F 1 "74HCT138" H 5100 2340 50  0000 C CNN
-F 2 "" H 5100 1650 50  0001 C CNN
+F 2 "Package_DIP:DIP-16_W7.62mm_Socket" H 5100 1650 50  0001 C CNN
 F 3 "" H 5100 1650 50  0001 C CNN
 	1    5100 1650
@@
 F 0 "U504" H 8150 5931 50  0000 C CNN
 F 1 "74HCT541" H 8150 5840 50  0000 C CNN
-F 2 "" H 8150 4950 50  0001 C CNN
+F 2 "Package_DIP:DIP-20_W7.62mm_Socket" H 8150 4950 50  0001 C CNN
 F 3 "" H 8150 4950 50  0001 C CNN
 	1    8150 4950
@@
 	4350 1550 4350 1600
 $Comp
-L power:GND #PWR?
+L power:GND #PWR0174
 U 1 1 5E444C89
 P 4350 1600
-F 0 "#PWR?" H 4350 1350 50  0001 C CNN
+F 0 "#PWR0174" H 4350 1350 50  0001 C CNN
 F 1 "GND" H 4355 1427 50  0000 C CNN
 F 2 "" H 4350 1600 50  0001 C CNN
@@
 	4100 1850 4100 1650
 $Comp
-L power:VCC #PWR?
+L power:VCC #PWR0175
 U 1 1 5E4564AB
 P 4100 1650
-F 0 "#PWR?" H 4100 1500 50  0001 C CNN
+F 0 "#PWR0175" H 4100 1500 50  0001 C CNN
 F 1 "VCC" H 4117 1823 50  0000 C CNN
 F 2 "" H 4100 1650 50  0001 C CNN
@@
 	5400 1050 5400 850
 $Comp
-L power:VCC #PWR?
+L power:VCC #PWR0176
 U 1 1 5E458D61
 P 5400 850
-F 0 "#PWR?" H 5400 700 50  0001 C CNN
+F 0 "#PWR0176" H 5400 700 50  0001 C CNN
 F 1 "VCC" H 5417 1023 50  0000 C CNN
 F 2 "" H 5400 850 50  0001 C CNN
@@
 	8450 1050 8450 800
 $Comp
-L power:VCC #PWR?
+L power:VCC #PWR0177
 U 1 1 5E45F8C2
 P 8450 800
-F 0 "#PWR?" H 8450 650 50  0001 C CNN
+F 0 "#PWR0177" H 8450 650 50  0001 C CNN
 F 1 "VCC" H 8467 973 50  0000 C CNN
 F 2 "" H 8450 800 50  0001 C CNN
@@
 	8500 4150 8500 3950
 $Comp
-L power:VCC #PWR?
+L power:VCC #PWR0178
 U 1 1 5E4645C6
 P 8500 3950
-F 0 "#PWR?" H 8500 3800 50  0001 C CNN
+F 0 "#PWR0178" H 8500 3800 50  0001 C CNN
 F 1 "VCC" H 8517 4123 50  0000 C CNN
 F 2 "" H 8500 3950 50  0001 C CNN
@@
 	8150 3050 8150 3200
 $Comp
-L power:GND #PWR?
+L power:GND #PWR0179
 U 1 1 5E46CD86
 P 8150 3200
-F 0 "#PWR?" H 8150 2950 50  0001 C CNN
+F 0 "#PWR0179" H 8150 2950 50  0001 C CNN
 F 1 "GND" H 8155 3027 50  0000 C CNN
 F 2 "" H 8150 3200 50  0001 C CNN
@@
 	8150 5750 8150 5900
 $Comp
-L power:GND #PWR?
+L power:GND #PWR0180
 U 1 1 5E46E409
 P 8150 5900
-F 0 "#PWR?" H 8150 5650 50  0001 C CNN
+F 0 "#PWR0180" H 8150 5650 50  0001 C CNN
 F 1 "GND" H 8155 5727 50  0000 C CNN
 F 2 "" H 8150 5900 50  0001 C CNN
@@
 	7500 5450 7500 5600
 $Comp
-L power:GND #PWR?
+L power:GND #PWR0181
 U 1 1 5E4A8020
 P 7500 5600
-F 0 "#PWR?" H 7500 5350 50  0001 C CNN
+F 0 "#PWR0181" H 7500 5350 50  0001 C CNN
 F 1 "GND" H 7505 5427 50  0000 C CNN
 F 2 "" H 7500 5600 50  0001 C CNN
@@
 	5100 2350 5100 2500
 $Comp
-L power:GND #PWR?
+L power:GND #PWR0182
 U 1 1 5E64FB23
 P 5100 2500
-F 0 "#PWR?" H 5100 2250 50  0001 C CNN
+F 0 "#PWR0182" H 5100 2250 50  0001 C CNN
 F 1 "GND" H 5105 2327 50  0000 C CNN
 F 2 "" H 5100 2500 50  0001 C CNN
@@
 	3200 3550 3200 2550
 $Comp
-L power:VCC #PWR?
+L power:VCC #PWR0183
 U 1 1 5E663AAB
 P 3200 2550
-F 0 "#PWR?" H 3200 2400 50  0001 C CNN
+F 0 "#PWR0183" H 3200 2400 50  0001 C CNN
 F 1 "VCC" H 3217 2723 50  0000 C CNN
 F 2 "" H 3200 2550 50  0001 C CNN
@@
 	3200 6550 3200 6700
 $Comp
-L power:GND #PWR?
+L power:GND #PWR0184
 U 1 1 5E67442E
 P 3200 6700
-F 0 "#PWR?" H 3200 6450 50  0001 C CNN
+F 0 "#PWR0184" H 3200 6450 50  0001 C CNN
 F 1 "GND" H 3205 6527 50  0000 C CNN
 F 2 "" H 3200 6700 50  0001 C CNN
@@
 	6950 2300 6950 2400
 $Comp
-L power:GND #PWR?
+L power:GND #PWR0185
 U 1 1 5ED0CA81
 P 6950 3200
-F 0 "#PWR?" H 6950 2950 50  0001 C CNN
+F 0 "#PWR0185" H 6950 2950 50  0001 C CNN
 F 1 "GND" H 6955 3027 50  0000 C CNN
 F 2 "" H 6950 3200 50  0001 C CNN
@@
 F 0 "C501" H 915 7046 50  0000 L CNN
 F 1 "0.1 μF" H 915 6955 50  0000 L CNN
-F 2 "" H 838 6850 50  0001 C CNN
+F 2 "Capacitor_THT:C_Disc_D5.0mm_W2.5mm_P2.50mm" H 838 6850 50  0001 C CNN
 F 3 "" H 800 7000 50  0001 C CNN
 	1    800  7000
@@
 F 0 "C502" H 1415 7046 50  0000 L CNN
 F 1 "0.1 μF" H 1415 6955 50  0000 L CNN
-F 2 "" H 1338 6850 50  0001 C CNN
+F 2 "Capacitor_THT:C_Disc_D5.0mm_W2.5mm_P2.50mm" H 1338 6850 50  0001 C CNN
 F 3 "" H 1300 7000 50  0001 C CNN
 	1    1300 7000
@@
 F 0 "C503" H 1915 7046 50  0000 L CNN
 F 1 "0.1 μF" H 1915 6955 50  0000 L CNN
-F 2 "" H 1838 6850 50  0001 C CNN
+F 2 "Capacitor_THT:C_Disc_D5.0mm_W2.5mm_P2.50mm" H 1838 6850 50  0001 C CNN
 F 3 "" H 1800 7000 50  0001 C CNN
 	1    1800 7000
@@
 F 0 "C504" H 2415 7046 50  0000 L CNN
 F 1 "0.1 μF" H 2415 6955 50  0000 L CNN
-F 2 "" H 2338 6850 50  0001 C CNN
+F 2 "Capacitor_THT:C_Disc_D5.0mm_W2.5mm_P2.50mm" H 2338 6850 50  0001 C CNN
 F 3 "" H 2300 7000 50  0001 C CNN
 	1    2300 7000
@@
 	1550 7400 1800 7400
 $Comp
-L power:VCC #PWR?
+L power:VCC #PWR0186
 U 1 1 5ED8CCE0
 P 1550 6500
-F 0 "#PWR?" H 1550 6350 50  0001 C CNN
+F 0 "#PWR0186" H 1550 6350 50  0001 C CNN
 F 1 "VCC" H 1567 6673 50  0000 C CNN
 F 2 "" H 1550 6500 50  0001 C CNN
@@
 $EndComp
 $Comp
-L power:GND #PWR?
+L power:GND #PWR0187
 U 1 1 5ED8CF8E
 P 1550 7550
-F 0 "#PWR?" H 1550 7300 50  0001 C CNN
+F 0 "#PWR0187" H 1550 7300 50  0001 C CNN
 F 1 "GND" H 1555 7377 50  0000 C CNN
 F 2 "" H 1550 7550 50  0001 C CNN
@@
 	9950 2500 9950 2200
 $Comp
-L power:VCC #PWR?
+L power:VCC #PWR0188
 U 1 1 5EDC1EFC
 P 9950 2200
-F 0 "#PWR?" H 9950 2050 50  0001 C CNN
+F 0 "#PWR0188" H 9950 2050 50  0001 C CNN
 F 1 "VCC" H 9967 2373 50  0000 C CNN
 F 2 "" H 9950 2200 50  0001 C CNN
@@
 F 0 "Y501" V 5700 3400 50  0000 R CNN
 F 1 "11.0592 MHz" V 5600 3700 50  0000 R CNN
-F 2 "" H 5650 3050 50  0001 C CNN
+F 2 "Crystal:Crystal_HC18-U_Vertical" H 5650 3050 50  0001 C CNN
 F 3 "" H 5650 3050 50  0001 C CNN
 	1    5650 3050
@@
 F 0 "C505" V 5950 2750 50  0000 C CNN
 F 1 "30pF" V 5950 3050 50  0000 C CNN
-F 2 "" H 6088 2750 50  0001 C CNN
+F 2 "Capacitor_THT:C_Disc_D3.8mm_W2.6mm_P2.50mm" H 6088 2750 50  0001 C CNN
 F 3 "" H 6050 2900 50  0001 C CNN
 	1    6050 2900
@@
 F 0 "C506" V 5950 3100 50  0000 C CNN
 F 1 "30pF" V 5950 3400 50  0000 C CNN
-F 2 "" H 6088 3100 50  0001 C CNN
+F 2 "Capacitor_THT:C_Disc_D3.8mm_W2.6mm_P2.50mm" H 6088 3100 50  0001 C CNN
 F 3 "" H 6050 3250 50  0001 C CNN
 	1    6050 3250
@@
 	6350 3250 6350 3400
 $Comp
-L power:GND #PWR?
+L power:GND #PWR0189
 U 1 1 5F09EB58
 P 6350 3400
-F 0 "#PWR?" H 6350 3150 50  0001 C CNN
+F 0 "#PWR0189" H 6350 3150 50  0001 C CNN
 F 1 "GND" H 6355 3227 50  0000 C CNN
 F 2 "" H 6350 3400 50  0001 C CNN
@@
 	1900 5750 1900 5550
 $Comp
-L power:VCC #PWR?
+L power:VCC #PWR0190
 U 1 1 5ED640C7
 P 1900 5550
-F 0 "#PWR?" H 1900 5400 50  0001 C CNN
+F 0 "#PWR0190" H 1900 5400 50  0001 C CNN
 F 1 "VCC" H 1917 5723 50  0000 C CNN
 F 2 "" H 1900 5550 50  0001 C CNN
@@
 F 0 "J501" H 768 3217 50  0000 C CNN
 F 1 "Conn_01x20" H 768 3126 50  0000 C CNN
-F 2 "" H 850 2100 50  0001 C CNN
+F 2 "Connector_PinHeader_2.54mm:PinHeader_1x20_P2.54mm_Vertical" H 850 2100 50  0001 C CNN
 F 3 "~" H 850 2100 50  0001 C CNN
 	1    850  2100
@@
 F 0 "J503" H 8718 675 50  0000 C CNN
 F 1 "Conn_01x02" H 8718 766 50  0000 C CNN
-F 2 "" H 8800 1000 50  0001 C CNN
+F 2 "Connector_PinHeader_2.54mm:PinHeader_1x02_P2.54mm_Vertical" H 8800 1000 50  0001 C CNN
 F 3 "~" H 8800 1000 50  0001 C CNN
 	1    8800 1000

Commit message: fix footprint for resistor network
Parts:
- RN501: footprint Resistors_THT:R_Array_SIP9 -> Resistor_THT:R_Array_SIP9
Changed lines of the file:
@@
 F 0 "RN501" V 2717 5350 50  0000 C CNN
 F 1 "R_Network08" V 2626 5350 50  0000 C CNN
-F 2 "Resistors_THT:R_Array_SIP9" V 2675 5350 50  0001 C CNN
+F 2 "Resistor_THT:R_Array_SIP9" V 2675 5350 50  0001 C CNN
 F 3 "" H 2200 5350 50  0001 C CNN
 	1    2200 5350
