File: HardwareDesign/CPUandGlueLogic.kicad_pcb (KiCad board)
At the start: 2 copper layers, 150 x 90 mm, 37 parts, among them J001 Conn_02x40_Odd_Even, J100 Conn_01x02, U101 74HCT245, U102 74HCT245, U103 74HCT245, U104 74HCT365, U105 MAX708, U106 HD6809, U107 74HCT00, U108 74HCT27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

Commit message: bugfix: GND and VCC were reversed on the backplane connector
Took the opportunity to fix other minor details on the
CPU and glue logic PCB, such as a missing component value
on the silkscreen, the pull-up resistors for the IRQ
inputs being too close to the backplane clip, and
the header for the external reset switch being a little
too close to the top of the board (insetting it a bit
is more appropriate if a right angle connector is
installed.)
Parts:
- moved R103 11.0 mm to (16.6, 5.90), turned to 270 degrees
- moved R102 9.17 mm to (14.3, 5.90), turned to 270 degrees
- moved R101 8.37 mm to (12.0, 5.90), turned to 270 degrees
- moved J100 3.70 mm to (86.0, 6.90)
- moved C106 2.10 mm to (13.5, 19.4), turned to 0 degrees
Connections:
- J001 pad 79: VCC -> GND
- J001 pad 80: GND -> VCC
Routing:
- net GND: track 811.4 -> 786.4 mm, vias 33 -> 34
- net VCC: track 626.4 -> 606.4 mm
- net Net-(J100-Pad2): track 32.2 -> 35.6 mm
- net Net-(R101-Pad2): track 7.14 -> 9.58 mm
- net /~IRQ: track 105.4 -> 106.5 mm, vias 1 -> 2
- net Net-(R103-Pad2): track 7.15 -> 8.12 mm
Other:
- board text added: "F68 6809 microcomputer CPU and glue logic module 8-Jun-2021"
- board text removed: "F68 6809 microcomputer CPU and glue logic module 20-May-2021"

Commit message: route ~IODEV0 through ~IODEV4 to backplane connector
For some reason, the pins of the 74HCT138 weren't labeled
with the same nets as the corresponding pins on the backplane
connector, even though they have continuity on the schematic.
Connections:
- U109 pad 11: /CPUandGlueLogic/~IODEV4~ -> /~IODEV4
- U109 pad 12: /CPUandGlueLogic/~IODEV3~ -> /~IODEV3
- U109 pad 13: /CPUandGlueLogic/~IODEV2~ -> /~IODEV2
- U109 pad 14: /CPUandGlueLogic/~IODEV1~ -> /~IODEV1
- U109 pad 15: /CPUandGlueLogic/~IODEV0~ -> /~IODEV0
Routing:
- net /~IODEV0: track 0.00 -> 50.0 mm, vias 0 -> 2
- net /~IODEV4: track 0.00 -> 43.4 mm
- net /~IODEV1: track 0.00 -> 42.9 mm
- net /~IODEV2: track 0.00 -> 42.7 mm
- net /~IODEV3: track 0.00 -> 42.6 mm
