File: HardwareDesign/Display.kicad_sch (KiCad schematic)
At the start: 37 parts, among them J601 Conn_01x12, U601 Upduino_3.0, U602 IDT7201, U603 74LVC245, U604 74LVC245

Commit message: prepare to create PCB for TMS9918A module
Parts:
- D601, D602, D603: footprint (none) -> LED_THT:LED_D5.0mm
- R625, R626, R627: footprint (none) -> Resistor_THT:R_Axial_DIN0207_L6.3mm_D2.5mm_P7.62mm_Horizontal
- U602: footprint (none) -> Package_DIP:DIP-28_W7.62mm_Socket
- U603, U604: footprint (none) -> Package_DIP:DIP-20_W7.62mm_Socket
Changed lines of the file:
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@@
     (property "Reference" "U602" (id 0) (at 125.73 146.5326 0))
     (property "Value" "IDT7201" (id 1) (at 125.73 148.844 0))
-    (property "Footprint" "" (id 2) (at 125.73 176.53 0)
+    (property "Footprint" "Package_DIP:DIP-28_W7.62mm_Socket" (id 2) (at 125.73 176.53 0)
       (effects (font (size 1.27 1.27)) hide)
     )
@@
     (property "Reference" "U603" (id 0) (at 214.63 117.729 0))
     (property "Value" "74LVC245" (id 1) (at 214.63 120.0404 0))
-    (property "Footprint" "" (id 2) (at 214.63 130.81 0)
+    (property "Footprint" "Package_DIP:DIP-20_W7.62mm_Socket" (id 2) (at 214.63 130.81 0)
       (effects (font (size 1.27 1.27)) hide)
     )
@@
     (property "Reference" "U604" (id 0) (at 214.63 153.289 0))
     (property "Value" "74LVC245" (id 1) (at 214.63 155.6004 0))
-    (property "Footprint" "" (id 2) (at 214.63 166.37 0)
+    (property "Footprint" "Package_DIP:DIP-20_W7.62mm_Socket" (id 2) (at 214.63 166.37 0)
       (effects (font (size 1.27 1.27)) hide)
     )
@@
   (symbol (lib_id "power:GND") (at 104.14 199.39 0) (unit 1)
     (in_bom yes) (on_board yes)
-    (property "Reference" "#PWR?" (id 0) (at 104.14 205.74 0)
+    (property "Reference" "#PWR0204" (id 0) (at 104.14 205.74 0)
       (effects (font (size 1.27 1.27)) hide)
     )
@@
   (symbol (lib_id "power:GND") (at 125.73 210.82 0) (unit 1)
     (in_bom yes) (on_board yes)
-    (property "Reference" "#PWR?" (id 0) (at 125.73 217.17 0)
+    (property "Reference" "#PWR0205" (id 0) (at 125.73 217.17 0)
       (effects (font (size 1.27 1.27)) hide)
     )
@@
   (symbol (lib_id "power:VCC") (at 71.12 124.46 0) (unit 1)
     (in_bom yes) (on_board yes)
-    (property "Reference" "#PWR?" (id 0) (at 71.12 128.27 0)
+    (property "Reference" "#PWR0208" (id 0) (at 71.12 128.27 0)
       (effects (font (size 1.27 1.27)) hide)
     )
@@
   (symbol (lib_id "power:VCC") (at 132.08 147.32 0) (unit 1)
     (in_bom yes) (on_board yes)
-    (property "Reference" "#PWR?" (id 0) (at 132.08 151.13 0)
+    (property "Reference" "#PWR0206" (id 0) (at 132.08 151.13 0)
       (effects (font (size 1.27 1.27)) hide)
     )
@@
   (symbol (lib_id "power:GND") (at 73.66 200.66 0) (unit 1)
     (in_bom yes) (on_board yes)
-    (property "Reference" "#PWR?" (id 0) (at 73.66 207.01 0)
+    (property "Reference" "#PWR0207" (id 0) (at 73.66 207.01 0)
       (effects (font (size 1.27 1.27)) hide)
     )
@@
   (symbol (lib_id "power:GND") (at 198.12 149.86 0) (unit 1)
     (in_bom yes) (on_board yes)
-    (property "Reference" "#PWR?" (id 0) (at 198.12 156.21 0)
+    (property "Reference" "#PWR0198" (id 0) (at 198.12 156.21 0)
       (effects (font (size 1.27 1.27)) hide)
     )
@@
   (symbol (lib_id "power:GND") (at 198.12 186.69 0) (unit 1)
     (in_bom yes) (on_board yes)
-    (property "Reference" "#PWR?" (id 0) (at 198.12 193.04 0)
+    (property "Reference" "#PWR0210" (id 0) (at 198.12 193.04 0)
       (effects (font (size 1.27 1.27)) hide)
     )
@@
   (symbol (lib_id "power:GND") (at 229.87 186.69 0) (unit 1)
     (in_bom yes) (on_board yes)
-    (property "Reference" "#PWR?" (id 0) (at 229.87 193.04 0)
+    (property "Reference" "#PWR0211" (id 0) (at 229.87 193.04 0)
       (effects (font (size 1.27 1.27)) hide)
     )
@@
   (symbol (lib_id "power:GND") (at 231.14 149.86 0) (unit 1)
     (in_bom yes) (on_board yes)
-    (property "Reference" "#PWR?" (id 0) (at 231.14 156.21 0)
+    (property "Reference" "#PWR0197" (id 0) (at 231.14 156.21 0)
       (effects (font (size 1.27 1.27)) hide)
     )
@@
   (symbol (lib_id "power:+3V3") (at 31.75 53.34 0) (unit 1)
     (in_bom yes) (on_board yes)
-    (property "Reference" "#PWR?" (id 0) (at 31.75 57.15 0)
+    (property "Reference" "#PWR0212" (id 0) (at 31.75 57.15 0)
       (effects (font (size 1.27 1.27)) hide)
     )
@@
   (symbol (lib_id "power:+3V3") (at 238.76 121.92 0) (unit 1)
     (in_bom yes) (on_board yes)
-    (property "Reference" "#PWR?" (id 0) (at 238.76 125.73 0)
+    (property "Reference" "#PWR0195" (id 0) (at 238.76 125.73 0)
       (effects (font (size 1.27 1.27)) hide)
     )
@@
   (symbol (lib_id "power:+3V3") (at 245.11 157.48 0) (unit 1)
     (in_bom yes) (on_board yes)
-    (property "Reference" "#PWR?" (id 0) (at 245.11 161.29 0)
+    (property "Reference" "#PWR0196" (id 0) (at 245.11 161.29 0)
       (effects (font (size 1.27 1.27)) hide)
     )
@@
   (symbol (lib_id "power:+3V3") (at 190.5 121.92 0) (unit 1)
     (in_bom yes) (on_board yes)
-    (property "Reference" "#PWR?" (id 0) (at 190.5 125.73 0)
+    (property "Reference" "#PWR0194" (id 0) (at 190.5 125.73 0)
       (effects (font (size 1.27 1.27)) hide)
     )
@@
   (symbol (lib_id "power:+3V3") (at 190.5 157.48 0) (unit 1)
     (in_bom yes) (on_board yes)
-    (property "Reference" "#PWR?" (id 0) (at 190.5 161.29 0)
+    (property "Reference" "#PWR0199" (id 0) (at 190.5 161.29 0)
       (effects (font (size 1.27 1.27)) hide)
     )
@@
   (symbol (lib_id "power:VCC") (at 147.32 140.97 0) (unit 1)
     (in_bom yes) (on_board yes)
-    (property "Reference" "#PWR?" (id 0) (at 147.32 144.78 0)
+    (property "Reference" "#PWR0203" (id 0) (at 147.32 144.78 0)
       (effects (font (size 1.27 1.27)) hide)
     )
@@
   (symbol (lib_id "power:VCC") (at 158.75 195.58 0) (unit 1)
     (in_bom yes) (on_board yes)
-    (property "Reference" "#PWR?" (id 0) (at 158.75 199.39 0)
+    (property "Reference" "#PWR0209" (id 0) (at 158.75 199.39 0)
       (effects (font (size 1.27 1.27)) hide)
     )
@@
     (property "Reference" "D601" (id 0) (at 137.16 73.66 0))
     (property "Value" "LED" (id 1) (at 143.51 72.39 0))
-    (property "Footprint" "" (id 2) (at 143.51 74.93 0)
+    (property "Footprint" "LED_THT:LED_D5.0mm" (id 2) (at 143.51 74.93 0)
       (effects (font (size 1.27 1.27)) hide)
     )
@@
     (property "Reference" "D602" (id 0) (at 137.16 78.74 0))
     (property "Value" "LED" (id 1) (at 143.51 77.47 0))
-    (property "Footprint" "" (id 2) (at 143.51 80.01 0)
+    (property "Footprint" "LED_THT:LED_D5.0mm" (id 2) (at 143.51 80.01 0)
       (effects (font (size 1.27 1.27)) hide)
     )
@@
     (property "Reference" "D603" (id 0) (at 137.16 83.82 0))
     (property "Value" "LED" (id 1) (at 143.51 82.55 0))
-    (property "Footprint" "" (id 2) (at 143.51 85.09 0)
+    (property "Footprint" "LED_THT:LED_D5.0mm" (id 2) (at 143.51 85.09 0)
       (effects (font (size 1.27 1.27)) hide)
     )
@@
     (property "Reference" "R625" (id 0) (at 121.92 73.66 90))
     (property "Value" "R" (id 1) (at 127 72.39 90))
-    (property "Footprint" "" (id 2) (at 127 73.152 90)
+    (property "Footprint" "Resistor_THT:R_Axial_DIN0207_L6.3mm_D2.5mm_P7.62mm_Horizontal" (id 2) (at 127 73.152 90)
       (effects (font (size 1.27 1.27)) hide)
     )
@@
     (property "Reference" "R626" (id 0) (at 121.92 78.74 90))
     (property "Value" "R" (id 1) (at 127 77.47 90))
-    (property "Footprint" "" (id 2) (at 127 78.232 90)
+    (property "Footprint" "Resistor_THT:R_Axial_DIN0207_L6.3mm_D2.5mm_P7.62mm_Horizontal" (id 2) (at 127 78.232 90)
       (effects (font (size 1.27 1.27)) hide)
     )
@@
     (property "Reference" "R627" (id 0) (at 121.92 83.82 90))
     (property "Value" "R" (id 1) (at 127 82.55 90))
-    (property "Footprint" "" (id 2) (at 127 83.312 90)
+    (property "Footprint" "Resistor_THT:R_Axial_DIN0207_L6.3mm_D2.5mm_P7.62mm_Horizontal" (id 2) (at 127 83.312 90)
       (effects (font (size 1.27 1.27)) hide)
     )
@@
   (symbol (lib_id "power:GND") (at 154.94 85.09 90) (unit 1)
     (in_bom yes) (on_board yes)
-    (property "Reference" "#PWR?" (id 0) (at 161.29 85.09 0)
-      (effects (font (size 1.27 1.27)) hide)
-    )
+    (property "Reference" "#PWR0213" (id 0) (at 161.29 85.09 0)
+      (effects (font (size 1.27 1.27)) hide)
+    )
