File: HardwareDesign/FPGADisplayController.kicad_sch (KiCad schematic)
At the start: 28 parts, among them J901 Conn_01x06, U901 SN74LVC245APW, U902 SN74LVC245APW, U903 SN74LVC245APW, U905 Upduino_3.0, U906 74HCT688, U907 74HCT32, U908 74LS574, Y904 25.175 MHz 7050 3.3V

Commit message: bank reg is 74HCT, not 74LS
Parts:
- U908: value 74LS574 -> 74HCT574
Changed lines of the file:
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@@
 			)
 		)
-		(property "Value" "74LS574"
+		(property "Value" "74HCT574"
 			(at 63.1033 121.92 0)
 			(effects

Commit message: HSync/VSync were reversed on FPGA & VGA connector
Connections:
- net HSync: now also U905.26 (GPIO46); no longer U905.27 (GPIO47)
- net VSync: now also U905.27 (GPIO47); no longer U905.26 (GPIO46)
Changed lines of the file:
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@@
 	(wire
 		(pts
-			(xy 281.94 119.38) (xy 281.94 184.15)
-		)
-		(stroke
-			(width 0)
-			(type default)
-		)
-	)
-	(wire
-		(pts
 			(xy 262.89 48.26) (xy 252.73 48.26)
 		)
@@
 	(wire
 		(pts
+			(xy 280.67 184.15) (xy 321.31 184.15)
+		)
+		(stroke
+			(width 0)
+			(type default)
+		)
+	)
+	(wire
+		(pts
 			(xy 19.05 114.3) (xy 29.21 114.3)
 		)
@@
 		)
 	)
+	(wire
+		(pts
+			(xy 281.94 119.38) (xy 281.94 186.69)
+		)
+		(stroke
+			(width 0)
+			(type default)
+		)
+	)
 	(bus
 		(pts
@@
 	(wire
 		(pts
-			(xy 280.67 186.69) (xy 321.31 186.69)
-		)
-		(stroke
-			(width 0)
-			(type default)
-		)
-	)
-	(wire
-		(pts
 			(xy 295.91 121.92) (xy 297.18 121.92)
 		)
@@
 	(wire
 		(pts
-			(xy 281.94 184.15) (xy 321.31 184.15)
-		)
-		(stroke
-			(width 0)
-			(type default)
-		)
-	)
-	(wire
-		(pts
 			(xy 109.22 218.44) (xy 119.38 218.44)
 		)
@@
 	(wire
 		(pts
-			(xy 280.67 121.92) (xy 280.67 186.69)
+			(xy 280.67 121.92) (xy 280.67 184.15)
 		)
 		(stroke
@@
 		)
 	)
+	(wire
+		(pts
+			(xy 281.94 186.69) (xy 321.31 186.69)
+		)
+		(stroke
+			(width 0)
+			(type default)
+		)
+	)
 	(bus
 		(pts
@@
 		)
 	)
+	(label "HSync"
+		(at 313.69 184.15 0)
+		(effects
+			(font
+				(size 1.27 1.27)
+			)
+			(justify left bottom)
+		)
+	)
 	(label "T~{R}"
 		(at 199.39 124.46 0)
@@
 	)
 	(label "VSync"
-		(at 261.62 121.92 0)
+		(at 261.62 119.38 0)
 		(effects
 			(font
@@
 	)
 	(label "HSync"
-		(at 261.62 119.38 0)
+		(at 261.62 121.92 0)
 		(effects
 			(font
@@
 		(effects
 			(font
+				(size 1.27 1.27)
+			)
+			(justify left bottom)
+		)
+	)
+	(label "VSync"
+		(at 313.69 186.69 0)
+		(effects
+			(font
