File: DisplayController/Pixgen.kicad_sch (KiCad schematic)
At the start: 11 parts, among them U601 GAL22V10, U602 74ACT574, U603 27SF512, U604 74ACT574, U605 GAL22V10

Commit message: fixed designators for decoupling caps
Parts:
- renumbered C1 to C601, C2 to C602, C3 to C603, C4 to C604, C5 to C605
Changed lines of the file:
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@@
 		(dnp no)
 		(fields_autoplaced yes)
-		(property "Reference" "C3"
+		(property "Reference" "C603"
 			(at 58.42 184.1499 0)
 			(effects
@@
 			(project "HW_VGA"
 				(path "/c4bd4b39-993a-4195-805f-b4de6fa4aea5/ada96480-51d2-4212-ac45-aae2a8a63ede"
-					(reference "C3")
+					(reference "C603")
 					(unit 1)
 				)
@@
 		(dnp no)
 		(fields_autoplaced yes)
-		(property "Reference" "C2"
+		(property "Reference" "C602"
 			(at 43.18 184.1499 0)
 			(effects
@@
 			(project "HW_VGA"
 				(path "/c4bd4b39-993a-4195-805f-b4de6fa4aea5/ada96480-51d2-4212-ac45-aae2a8a63ede"
-					(reference "C2")
+					(reference "C602")
 					(unit 1)
 				)
@@
 		(dnp no)
 		(fields_autoplaced yes)
-		(property "Reference" "C4"
+		(property "Reference" "C604"
 			(at 73.66 184.1499 0)
 			(effects
@@
 			(project "HW_VGA"
 				(path "/c4bd4b39-993a-4195-805f-b4de6fa4aea5/ada96480-51d2-4212-ac45-aae2a8a63ede"
-					(reference "C4")
+					(reference "C604")
 					(unit 1)
 				)
@@
 		(dnp no)
 		(fields_autoplaced yes)
-		(property "Reference" "C1"
+		(property "Reference" "C601"
 			(at 27.94 184.1499 0)
 			(effects
@@
 			(project "HW_VGA"
 				(path "/c4bd4b39-993a-4195-805f-b4de6fa4aea5/ada96480-51d2-4212-ac45-aae2a8a63ede"
-					(reference "C1")
+					(reference "C601")
 					(unit 1)
 				)
@@
 		(dnp no)
 		(fields_autoplaced yes)
-		(property "Reference" "C5"
+		(property "Reference" "C605"
 			(at 88.9 184.1499 0)
 			(effects
@@
 			(project "HW_VGA"
 				(path "/c4bd4b39-993a-4195-805f-b4de6fa4aea5/ada96480-51d2-4212-ac45-aae2a8a63ede"
-					(reference "C5")
-					(unit 1)
-				)
+					(reference "C605")
+					(unit 1)
+				)

Commit message: assigned footprints
Will need to double check.
Parts:
- C601, C602, C603, C604, C605: footprint (none) -> Capacitor_SMD:C_0805_2012Metric_Pad1.18x1.45mm_HandSolder
- R601: footprint (none) -> Resistor_SMD:R_0805_2012Metric_Pad1.20x1.40mm_HandSolder
- U601, U605: footprint (none) -> Package_DIP:DIP-24_W7.62mm_Socket
- U602, U604: footprint (none) -> Package_SO:SOIC-20W_7.5x12.8mm_P1.27mm
- U603: footprint MODULE -> Package_DIP:DIP-28_W15.24mm_Socket
Changed lines of the file:
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@@
 			)
 		)
-		(property "Footprint" ""
+		(property "Footprint" "Capacitor_SMD:C_0805_2012Metric_Pad1.18x1.45mm_HandSolder"
 			(at 55.5752 189.23 0)
 			(effects
@@
 			)
 		)
-		(property "Footprint" ""
+		(property "Footprint" "Capacitor_SMD:C_0805_2012Metric_Pad1.18x1.45mm_HandSolder"
 			(at 40.3352 189.23 0)
 			(effects
@@
 			)
 		)
-		(property "Footprint" ""
+		(property "Footprint" "Resistor_SMD:R_0805_2012Metric_Pad1.20x1.40mm_HandSolder"
 			(at 130.302 35.56 90)
 			(effects
@@
 			)
 		)
-		(property "Footprint" ""
+		(property "Footprint" "Package_SO:SOIC-20W_7.5x12.8mm_P1.27mm"
 			(at 77.47 77.47 0)
 			(effects
@@
 			)
 		)
-		(property "Footprint" "MODULE"
+		(property "Footprint" "Package_DIP:DIP-28_W15.24mm_Socket"
 			(at 154.94 58.42 0)
 			(effects
@@
 			)
 		)
-		(property "Footprint" ""
+		(property "Footprint" "Package_DIP:DIP-24_W7.62mm_Socket"
 			(at 227.33 102.87 0)
 			(effects
@@
 			)
 		)
-		(property "Footprint" ""
+		(property "Footprint" "Package_DIP:DIP-24_W7.62mm_Socket"
 			(at 153.67 138.43 0)
 			(effects
@@
 			)
 		)
-		(property "Footprint" ""
+		(property "Footprint" "Capacitor_SMD:C_0805_2012Metric_Pad1.18x1.45mm_HandSolder"
 			(at 70.8152 189.23 0)
 			(effects
@@
 			)
 		)
-		(property "Footprint" ""
+		(property "Footprint" "Capacitor_SMD:C_0805_2012Metric_Pad1.18x1.45mm_HandSolder"
 			(at 25.0952 189.23 0)
 			(effects
@@
 			)
 		)
-		(property "Footprint" ""
+		(property "Footprint" "Capacitor_SMD:C_0805_2012Metric_Pad1.18x1.45mm_HandSolder"
 			(at 86.0552 189.23 0)
 			(effects
@@
 			)
 		)
-		(property "Footprint" ""
+		(property "Footprint" "Package_SO:SOIC-20W_7.5x12.8mm_P1.27mm"
 			(at 63.5 137.16 0)
 			(effects

Commit message: initial PCB component placement
Changed package for GAL22V10 to SOIC24 rather than DIP24.
That means we'll use ATF22V10C parts (which are available
as SOIC24.)

Now for the routing :-)
Parts:
- U601, U605: footprint Package_DIP:DIP-24_W7.62mm_Socket -> Package_SO:SOIC-24W_7.5x15.4mm_P1.27mm
Changed lines of the file:
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@@
 			)
 		)
-		(property "Footprint" "Package_DIP:DIP-24_W7.62mm_Socket"
+		(property "Footprint" "Package_SO:SOIC-24W_7.5x15.4mm_P1.27mm"
 			(at 227.33 102.87 0)
 			(effects
@@
 			)
 		)
-		(property "Footprint" "Package_DIP:DIP-24_W7.62mm_Socket"
+		(property "Footprint" "Package_SO:SOIC-24W_7.5x15.4mm_P1.27mm"
 			(at 153.67 138.43 0)
 			(effects
