File: DisplayController/VRAM.kicad_sch (KiCad schematic)
At the start: 8 parts, among them U801 IDT7134, U802 IDT7134, U803 GAL22V10, U804 74HCT574

Commit message: assigned footprints
Will need to double check.
Parts:
- C801, C802, C803, C804: footprint (none) -> Capacitor_SMD:C_0805_2012Metric_Pad1.18x1.45mm_HandSolder
- U801, U802: footprint MODULE -> Package_LCC:PLCC-52_THT-Socket
- U803: footprint (none) -> Package_DIP:DIP-24_W7.62mm_Socket
- U804: footprint (none) -> Package_LCC:PLCC-52_THT-Socket
Changed lines of the file:
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@@
 			)
 		)
-		(property "Footprint" ""
+		(property "Footprint" "Capacitor_SMD:C_0805_2012Metric_Pad1.18x1.45mm_HandSolder"
 			(at 83.5152 199.39 0)
 			(effects
@@
 			)
 		)
-		(property "Footprint" ""
+		(property "Footprint" "Capacitor_SMD:C_0805_2012Metric_Pad1.18x1.45mm_HandSolder"
 			(at 37.7952 199.39 0)
 			(effects
@@
 			)
 		)
-		(property "Footprint" ""
+		(property "Footprint" "Package_LCC:PLCC-52_THT-Socket"
 			(at 86.36 48.26 0)
 			(effects
@@
 			)
 		)
-		(property "Footprint" "MODULE"
+		(property "Footprint" "Package_LCC:PLCC-52_THT-Socket"
 			(at 232.41 165.1 0)
 			(effects
@@
 			)
 		)
-		(property "Footprint" ""
+		(property "Footprint" "Capacitor_SMD:C_0805_2012Metric_Pad1.18x1.45mm_HandSolder"
 			(at 53.0352 199.39 0)
 			(effects
@@
 			)
 		)
-		(property "Footprint" "MODULE"
+		(property "Footprint" "Package_LCC:PLCC-52_THT-Socket"
 			(at 232.41 69.85 0)
 			(effects
@@
 			)
 		)
-		(property "Footprint" ""
+		(property "Footprint" "Package_DIP:DIP-24_W7.62mm_Socket"
 			(at 100.33 127 0)
 			(effects
@@
 			)
 		)
-		(property "Footprint" ""
+		(property "Footprint" "Capacitor_SMD:C_0805_2012Metric_Pad1.18x1.45mm_HandSolder"
 			(at 68.2752 199.39 0)
 			(effects

Commit message: fixed another incorrect footprint assignment
Parts:
- U804: footprint Package_LCC:PLCC-52_THT-Socket -> Package_SO:SOIC-20W_7.5x12.8mm_P1.27mm
Changed lines of the file:
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@@
 			)
 		)
-		(property "Footprint" "Package_LCC:PLCC-52_THT-Socket"
+		(property "Footprint" "Package_SO:SOIC-20W_7.5x12.8mm_P1.27mm"
 			(at 86.36 48.26 0)
 			(effects

Commit message: initial PCB component placement
Changed package for GAL22V10 to SOIC24 rather than DIP24.
That means we'll use ATF22V10C parts (which are available
as SOIC24.)

Now for the routing :-)
Parts:
- U803: footprint Package_DIP:DIP-24_W7.62mm_Socket -> Package_SO:SOIC-24W_7.5x15.4mm_P1.27mm
Changed lines of the file:
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@@
 			)
 		)
-		(property "Footprint" "Package_DIP:DIP-24_W7.62mm_Socket"
+		(property "Footprint" "Package_SO:SOIC-24W_7.5x15.4mm_P1.27mm"
 			(at 100.33 127 0)
 			(effects
